File: led1.kicad_sch (KiCad schematic)
At the start: 0 parts

Commit message: led + resistor + 5v
Parts:
- added D1: LED, symbol Device:LED
- added R1: R, symbol Device:R
Connections:
- new net: D1.2 (A), R1.1
- new net +5V: D1.1 (K)
- new net GND: R1.2
Other:
- note added: "LED SIMPLE"
- company: (none) -> DR SYSTEMS 
- title: (none) -> LED 
